Commit message: clober_gazebo 추가

File: clober_description/urdf/clober.urdf.xacro (robot description, xacro)
@@ -84,3 +84,87 @@
     <origin xyz="0.159 0 0.2265" rpy="3.1415926535897931 0 0"/>
   </xacro:sensor_tim571> -->
+  <joint name="caster_joint1" type="continuous">
+    <parent link="base_link"/>
+    <child link="caster_link1"/>
+    <origin xyz="0.11 0.13 -0.04" rpy="1.5707963267948966 0 0"/>
+    <axis xyz="0 0 1" rpy="0 0 0"/>
+  </joint>
+  <link name="caster_link1">
+    <collision>
+      <origin xyz="0 0 0" rpy="0 0 0"/>
+      <geometry>
+        <cylinder length="0.02" radius="0.025"/>
+      </geometry>
+    </collision>
+    <inertial>
+      <origin xyz="0 0 0" />
+      <mass value="0.005" />
+      <inertia ixx="0.001" ixy="0.0" ixz="0.0"
+               iyy="0.001" iyz="0.0"
+               izz="0.001" />
+    </inertial>
+  </link>
+  <joint name="caster_joint2" type="continuous">
+    <parent link="base_link"/>
+    <child link="caster_link2"/>
+    <origin xyz="-0.11 0.13 -0.04" rpy="1.5707963267948966 0 0"/>
+    <axis xyz="0 0 1" rpy="0 0 0"/>
+  </joint>
+  <link name="caster_link2">
+    <collision>
+      <origin xyz="0 0 0" rpy="0 0 0"/>
+      <geometry>
+        <cylinder length="0.02" radius="0.025"/>
+      </geometry>
+    </collision>
+    <inertial>
+      <origin xyz="0 0 0" />
+      <mass value="0.005" />
+      <inertia ixx="0.001" ixy="0.0" ixz="0.0"
+               iyy="0.001" iyz="0.0"
+               izz="0.001" />
+    </inertial>
+  </link>
+  <joint name="caster_joint3" type="continuous">
+    <parent link="base_link"/>
+    <child link="caster_link3"/>
+    <origin xyz="0.11 -0.13 -0.04" rpy="1.5707963267948966 0 0"/>
+    <axis xyz="0 0 1" rpy="0 0 0"/>
+  </joint>
+  <link name="caster_link3">
+    <collision>
+      <origin xyz="0 0 0" rpy="0 0 0"/>
+      <geometry>
+        <cylinder length="0.02" radius="0.025"/>
+      </geometry>
+    </collision>
+    <inertial>
+      <origin xyz="0 0 0" />
+      <mass value="0.005" />
+      <inertia ixx="0.001" ixy="0.0" ixz="0.0"
+               iyy="0.001" iyz="0.0"
+               izz="0.001" />
+    </inertial>
+  </link>
+  <joint name="caster_joint4" type="continuous">
+    <parent link="base_link"/>
+    <child link="caster_link4"/>
+    <origin xyz="-0.11 -0.13 -0.04" rpy="1.5707963267948966 0 0"/>
+    <axis xyz="0 0 1" rpy="0 0 0"/>
+  </joint>
+  <link name="caster_link4">
+    <collision>
+      <origin xyz="0 0 0" rpy="0 0 0"/>
+      <geometry>
+        <cylinder length="0.02" radius="0.025"/>
+      </geometry>
+    </collision>
+    <inertial>
+      <origin xyz="0 0 0" />
+      <mass value="0.005" />
+      <inertia ixx="0.001" ixy="0.0" ixz="0.0"
+               iyy="0.001" iyz="0.0"
+               izz="0.001" />
+    </inertial>
+  </link>
 </robot>

Commit message: clober slam navigation launch

File: clober_description/urdf/clober.urdf.xacro (robot description, xacro)
@@ -77,8 +77,8 @@
   <joint name="lidar_joint" type="fixed">
     <parent link="base_link"/>
-    <child link="lidar_link"/>
+    <child link="laser_link"/>
     <origin xyz="0.159 0 0.2265" rpy="3.1415926535897931 0 0"/>
   </joint>
-  <link name="lidar_link"/>
+  <link name="laser_link"/>
   <!-- <xacro:sensor_tim571 parent="base_link">
     <origin xyz="0.159 0 0.2265" rpy="3.1415926535897931 0 0"/>

Commit message: modified urdf.xacro file for base_link size

File: clober_description/urdf/clober.urdf.xacro (robot description, xacro)
@@ -21,7 +21,7 @@
         </visual>
         <collision>
-            <origin xyz="0 0 0.2" rpy="0 0 ${PI/2}"/>
-            <geometry>
-                <box size="0.5 0.5 0.3"/>
+            <origin xyz="0 0 0.05" rpy="0 0 ${PI/2}"/>
+            <geometry>
+                <box size="0.41 0.41 0.1"/>
             </geometry>
         </collision>
@@ -197,9 +197,10 @@
         <parent link="base_link"/>
         <child link="base_scan"/>
-        <origin xyz="0.159 0 0.4" rpy="${PI} 0 0"/>
-    </joint>
+        <origin xyz="0.159 0 0.16" rpy="${PI} 0 0"/>
+    </joint>
+    <!-- <origin xyz="0.21 0 0.16" rpy="${PI} 0 0"/> -->
     <link name="base_scan">
       <visual>
-          <origin xyz="0 0 0.2265"    rpy="0 0 0"/>
+          <origin xyz="0 0 0.0"    rpy="0 0 0"/>
           <geometry>
               <mesh filename="package://clober_description/meshes/include/tim571.stl"/>

Commit message: add gmapping launch

File: clober_description/urdf/clober.urdf.xacro (robot description, xacro)
@@ -78,5 +78,5 @@
     <parent link="base_link"/>
     <child link="laser_link"/>
-    <origin xyz="0.159 0 0.2265" rpy="3.1415926535897931 0 0"/>
+    <origin xyz="0.159 0 0.2265" rpy="0 0 0"/>
   </joint>
   <link name="laser_link"/>

Commit message: update

File: clober_description/urdf/clober.urdf.xacro (robot description, xacro)
@@ -202,5 +202,5 @@
     <link name="base_scan">
       <visual>
-          <origin xyz="0 0 0.0"    rpy="0 0 0"/>
+          <origin xyz="0 0 0"    rpy="0 0 0"/>
           <geometry>
               <mesh filename="package://clober_description/meshes/include/tim571.stl"/>

Commit message: add ekf and modify clober_serial with myahrs_ros2_driver

File: clober_description/urdf/clober.urdf.xacro (robot description, xacro)
@@ -3,4 +3,10 @@
   <!-- <xacro:include filename="$(find clober_description)/urdf/include/tim571.urdf.xacro"/> -->
   <xacro:property name="PI" value="3.1415926535897931"/>
+  <link name="base_footprint"/>
+  <joint name="base_joint" type="fixed">
+      <parent link="base_footprint"/>
+      <child link="base_link"/>
+      <origin xyz="0.0 0.0 0.020" rpy="0 0 0"/>
+  </joint>
   <link name="base_link">
     <visual>

Commit message: add temporary test file

File: clober_description/urdf/clober.urdf.xacro (robot description, xacro)
@@ -179,5 +179,6 @@
         <parent link="base_link"/>
         <child link="imu_link"/>
-        <origin xyz="0.0605 0 0.0923" rpy="0 0 0"/>
+        <origin xyz="0.15 0 0.225" rpy="0 0 0"/>
+        <!-- <origin xyz="0.0605 0 0.0923" rpy="0 0 0"/> -->
     </joint>
     <link name="imu_link"/>

Commit message: add tc version

File: clober_description/urdf/clober.urdf.xacro (robot description, xacro)
@@ -7,11 +7,11 @@
     <xacro:include filename="$(find clober_description)/urdf/clober.gazebo.xacro"/>
     <xacro:property name="PI" value="3.1415926535897931"/>
-    <link name="base_footprint"/>
-    <joint name="base_joint" type="fixed">
-        <parent link="base_footprint"/>
-        <child link="base_link"/>
+    <link name="$(arg prefix)base_footprint"/>
+    <joint name="$(arg prefix)base_joint" type="fixed">
+        <parent link="$(arg prefix)base_footprint"/>
+        <child link="$(arg prefix)base_link"/>
         <origin xyz="0.0 0.0 0.020" rpy="0 0 0"/>
     </joint>
-    <link name="base_link">
+    <link name="$(arg prefix)base_link">
         <visual>
             <origin xyz="0 0 0" rpy="0 0 ${PI/2}"/>
@@ -38,11 +38,11 @@
         </inertial>
     </link>
-    <joint name="wheel_left_joint" type="continuous">
-        <parent link="base_link"/>
-        <child link="wheel_left_link"/>
+    <joint name="$(arg prefix)wheel_left_joint" type="continuous">
+        <parent link="$(arg prefix)base_link"/>
+        <child link="$(arg prefix)wheel_left_link"/>
         <origin xyz="0.0018 0.1558 0.02" rpy="0 0 0"/>
         <axis xyz="0 1 0" rpy="0 0 0"/>
     </joint>
-    <link name="wheel_left_link">
+    <link name="$(arg prefix)wheel_left_link">
         <visual>
             <origin xyz="0 0 0" rpy="0 0 -${PI/2}"/>
@@ -69,11 +69,11 @@
         </inertial>
     </link>
-    <joint name="wheel_right_joint" type="continuous">
-        <parent link="base_link"/>
-        <child link="wheel_right_link"/>
+    <joint name="$(arg prefix)wheel_right_joint" type="continuous">
+        <parent link="$(arg prefix)base_link"/>
+        <child link="$(arg prefix)wheel_right_link"/>
         <origin xyz="0.0018 -0.1558 0.02" rpy="0 0 0"/>
         <axis xyz="0 1 0" rpy="0 0 0"/>
     </joint>
-    <link name="wheel_right_link">
+    <link name="$(arg prefix)wheel_right_link">
         <visual>
             <origin xyz="0 0 0" rpy="0 0 ${PI/2}"/>
@@ -100,106 +100,106 @@
         </inertial>
     </link>
-    <joint name="caster_joint1" type="continuous">
-        <parent link="base_link"/>
-        <child link="caster_link1"/>
+    <joint name="$(arg prefix)caster_joint1" type="continuous">
+        <parent link="$(arg prefix)base_link"/>
+        <child link="$(arg prefix)caster_link1"/>
         <origin xyz="0.11 0.13 -0.04" rpy="${PI/2} 0 0"/>
         <axis xyz="0 0 1" rpy="0 0 0"/>
     </joint>
-    <link name="caster_link1">
-        <collision>
-            <origin xyz="0 0 0" rpy="0 0 0"/>
-            <geometry>
-                <cylinder length="0.02" radius="0.025"/>
-            </geometry>
-        </collision>
-        <inertial>
-            <origin xyz="0 0 0"/>
-            <mass value="0.005"/>
-            <inertia ixx="0.001" ixy="0.0" ixz="0.0" iyy="0.001" iyz="0.0" izz="0.001"/>
-        </inertial>
-    </link>
-    <joint name="caster_joint2" type="continuous">
-        <parent link="base_link"/>
-        <child link="caster_link2"/>
+    <link name="$(arg prefix)caster_link1">
+        <collision>
+            <origin xyz="0 0 0" rpy="0 0 0"/>
+            <geometry>
+                <cylinder length="0.02" radius="0.025"/>
+            </geometry>
+        </collision>
+        <inertial>
+            <origin xyz="0 0 0"/>
+            <mass value="0.005"/>
+            <inertia ixx="0.001" ixy="0.0" ixz="0.0" iyy="0.001" iyz="0.0" izz="0.001"/>
+        </inertial>
+    </link>
+    <joint name="$(arg prefix)caster_joint2" type="continuous">
+        <parent link="$(arg prefix)base_link"/>
+        <child link="$(arg prefix)caster_link2"/>
         <origin xyz="-0.11 0.13 -0.04" rpy="${PI/2} 0 0"/>
         <axis xyz="0 0 1" rpy="0 0 0"/>
     </joint>
-    <link name="caster_link2">
-        <collision>
-            <origin xyz="0 0 0" rpy="0 0 0"/>
-            <geometry>
-                <cylinder length="0.02" radius="0.025"/>
-            </geometry>
-        </collision>
-        <inertial>
-            <origin xyz="0 0 0"/>
-            <mass value="0.005"/>
-            <inertia ixx="0.001" ixy="0.0" ixz="0.0" iyy="0.001" iyz="0.0" izz="0.001"/>
-        </inertial>
-    </link>
-    <joint name="caster_joint3" type="continuous">
-        <parent link="base_link"/>
-        <child link="caster_link3"/>
+    <link name="$(arg prefix)caster_link2">
+        <collision>
+            <origin xyz="0 0 0" rpy="0 0 0"/>
+            <geometry>
+                <cylinder length="0.02" radius="0.025"/>
+            </geometry>
+        </collision>
+        <inertial>
+            <origin xyz="0 0 0"/>
+            <mass value="0.005"/>
+            <inertia ixx="0.001" ixy="0.0" ixz="0.0" iyy="0.001" iyz="0.0" izz="0.001"/>
+        </inertial>
+    </link>
+    <joint name="$(arg prefix)caster_joint3" type="continuous">
+        <parent link="$(arg prefix)base_link"/>
+        <child link="$(arg prefix)caster_link3"/>
         <origin xyz="0.11 -0.13 -0.04" rpy="${PI/2} 0 0"/>
         <axis xyz="0 0 1" rpy="0 0 0"/>
     </joint>
-    <link name="caster_link3">
-        <collision>
-            <origin xyz="0 0 0" rpy="0 0 0"/>
-            <geometry>
-                <cylinder length="0.02" radius="0.025"/>
-            </geometry>
-        </collision>
-        <inertial>
-            <origin xyz="0 0 0"/>
-            <mass value="0.005"/>
-            <inertia ixx="0.001" ixy="0.0" ixz="0.0" iyy="0.001" iyz="0.0" izz="0.001"/>
-        </inertial>
-    </link>
-    <joint name="caster_joint4" type="continuous">
-        <parent link="base_link"/>
-        <child link="caster_link4"/>
+    <link name="$(arg prefix)caster_link3">
+        <collision>
+            <origin xyz="0 0 0" rpy="0 0 0"/>
+            <geometry>
+                <cylinder length="0.02" radius="0.025"/>
+            </geometry>
+        </collision>
+        <inertial>
+            <origin xyz="0 0 0"/>
+            <mass value="0.005"/>
+            <inertia ixx="0.001" ixy="0.0" ixz="0.0" iyy="0.001" iyz="0.0" izz="0.001"/>
+        </inertial>
+    </link>
+    <joint name="$(arg prefix)caster_joint4" type="continuous">
+        <parent link="$(arg prefix)base_link"/>
+        <child link="$(arg prefix)caster_link4"/>
         <origin xyz="-0.11 -0.13 -0.04" rpy="${PI/2} 0 0"/>
         <axis xyz="0 0 1" rpy="0 0 0"/>
     </joint>
-    <link name="caster_link4">
-        <collision>
-            <origin xyz="0 0 0" rpy="0 0 0"/>
-            <geometry>
-                <cylinder length="0.02" radius="0.025"/>
-            </geometry>
-        </collision>
-        <inertial>
-            <origin xyz="0 0 0"/>
-            <mass value="0.005"/>
-            <inertia ixx="0.001" ixy="0.0" ixz="0.0" iyy="0.001" iyz="0.0" izz="0.001"/>
-        </inertial>
-    </link>
-    <joint name="imu_joint" type="fixed">
-        <parent link="base_link"/>
-        <child link="imu_link"/>
+    <link name="$(arg prefix)caster_link4">
+        <collision>
+            <origin xyz="0 0 0" rpy="0 0 0"/>
+            <geometry>
+                <cylinder length="0.02" radius="0.025"/>
+            </geometry>
+        </collision>
+        <inertial>
+            <origin xyz="0 0 0"/>
+            <mass value="0.005"/>
+            <inertia ixx="0.001" ixy="0.0" ixz="0.0" iyy="0.001" iyz="0.0" izz="0.001"/>
+        </inertial>
+    </link>
+    <joint name="$(arg prefix)imu_joint" type="fixed">
+        <parent link="$(arg prefix)base_link"/>
+        <child link="$(arg prefix)imu_link"/>
         <origin xyz="0.15 0 0.225" rpy="0 0 0"/>
         <!-- <origin xyz="0.0605 0 0.0923" rpy="0 0 0"/> -->
     </joint>
-    <link name="imu_link"/>
-    <joint name="left_ultrasonic_joint" type="fixed">
-        <parent link="base_link"/>
-        <child link="left_ultrasonic"/>
+    <link name="$(arg prefix)imu_link"/>
+    <joint name="$(arg prefix)left_ultrasonic_joint" type="fixed">
+        <parent link="$(arg prefix)base_link"/>
+        <child link="$(arg prefix)left_ultrasonic"/>
         <origin xyz="0.18164 0.09679 0.08396" rpy="0 0 0"/>
     </joint>
-    <link name="left_ultrasonic"/>
-    <joint name="right_ultrasonic_joint" type="fixed">
-        <parent link="base_link"/>
-        <child link="right_ultrasonic"/>
+    <link name="$(arg prefix)left_ultrasonic"/>
+    <joint name="$(arg prefix)right_ultrasonic_joint" type="fixed">
+        <parent link="$(arg prefix)base_link"/>
+        <child link="$(arg prefix)right_ultrasonic"/>
         <origin xyz="0.18164 -0.09679 0.08396" rpy="0 0 0"/>
     </joint>
-    <link name="right_ultrasonic"/>
-    <joint name="base_scan_joint" type="fixed">
-        <parent link="base_link"/>
-        <child link="base_scan"/>
+    <link name="$(arg prefix)right_ultrasonic"/>
+    <joint name="$(arg prefix)base_scan_joint" type="fixed">
+        <parent link="$(arg prefix)base_link"/>
+        <child link="$(arg prefix)base_scan"/>
         <origin xyz="0.159 0 0.16" rpy="${PI} 0 0"/>
     </joint>
     <!-- <origin xyz="0.21 0 0.16" rpy="${PI} 0 0"/> -->
-    <link name="base_scan">
+    <link name="$(arg prefix)base_scan">
       <visual>
           <origin xyz="0 0 0"    rpy="0 0 0"/>
@@ -211,6 +211,6 @@
     <!-- <xacro:sensor_tim571 parent="base_link"> <origin xyz="0.159 0 0.2265"
     rpy="${PI} 0 0"/> </xacro:sensor_tim571> -->
-    <xacro:sensor_d435 parent="base_link" name="camera">
+    <!-- <xacro:sensor_d435 parent="$(arg prefix)base_link" name="camera">
         <origin xyz="0.17573 0 0.06791" rpy="0 -${PI/12} 0"/>
-    </xacro:sensor_d435>
+    </xacro:sensor_d435> -->
 </robot>

Commit message: update urdf files

File: clober_description/urdf/clober.urdf.xacro (robot description, xacro)
@@ -179,6 +179,5 @@
         <parent link="$(arg prefix)base_link"/>
         <child link="$(arg prefix)imu_link"/>
-        <origin xyz="0.15 0 0.225" rpy="0 0 0"/>
-        <!-- <origin xyz="0.0605 0 0.0923" rpy="0 0 0"/> -->
+        <origin xyz="0.0605 0 0.0923" rpy="0 0 0"/>
     </joint>
     <link name="$(arg prefix)imu_link"/>
@@ -211,6 +210,6 @@
     <!-- <xacro:sensor_tim571 parent="base_link"> <origin xyz="0.159 0 0.2265"
     rpy="${PI} 0 0"/> </xacro:sensor_tim571> -->
-    <!-- <xacro:sensor_d435 parent="$(arg prefix)base_link" name="camera">
+    <xacro:sensor_d435 parent="$(arg prefix)base_link" name="$(arg prefix)camera">
         <origin xyz="0.17573 0 0.06791" rpy="0 -${PI/12} 0"/>
-    </xacro:sensor_d435> -->
+    </xacro:sensor_d435>
 </robot>

Commit message: [chore]: Add suntech office launch file for simulation
- Add 3-clobers param

File: clober_description/urdf/clober.urdf.xacro (robot description, xacro)
@@ -21,7 +21,7 @@
         </visual>
         <collision>
-            <origin xyz="0 0 0.05" rpy="0 0 ${PI/2}"/>
-            <geometry>
-                <box size="0.41 0.41 0.1"/>
+            <origin xyz="0 0 0.02" rpy="0 0 ${PI/2}"/>
+            <geometry>
+                <mesh filename="package://clober_description/meshes/clober.dae"/>
             </geometry>
         </collision>
